File: hardware/light_board/light_board.kicad_pcb (KiCad board)
At the start: 2 copper layers, 24 x 24 mm, 11 parts, among them J1 LED 1 -, J2 LED 2 -, J3 Conn_01x06_Socket, J4 LED 1 +, J5 LED 2 +

Commit message: add sponsor to PCBs
Signed-off-by: Peter Siegmund <mars3142@users.noreply.github.com>
Parts:
- added G***: LOGO, LOGO, F.Cu at (100.2, 51.8)
- R1, R2: value 100R -> 1K
