File: hardware/light_board/light_board.kicad_pcb (KiCad board)
At the start: 2 copper layers, 24 x 24 mm, 12 parts, among them J1 LED 1 -, J2 LED 2 -, J3 Conn_01x06_Socket, J4 LED 1 +, J5 LED 2 +

Commit message: latest KiCad changes
Signed-off-by: Peter Siegmund <mars3142@users.noreply.github.com>
Connections:
- net BEACON renamed /BEACON
- net OUTDOOR_L renamed /OUTDOOR_L
- net OUTDOOR_R renamed /OUTDOOR_R
Changed lines of the file:
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@@
 	(net 0 "")
 	(net 1 "GND")
-	(net 2 "BEACON")
+	(net 2 "/BEACON")
 	(net 3 "+5V")
 	(net 4 "unconnected-(D1-DOUT-Pad2)")
-	(net 5 "OUTDOOR_L")
-	(net 6 "OUTDOOR_R")
+	(net 5 "/OUTDOOR_L")
+	(net 6 "/OUTDOOR_R")
 	(net 7 "Net-(J4-Pad1)")
 	(net 8 "Net-(J5-Pad1)")
@@
 			(layers "F.Cu" "F.Mask" "F.Paste")
 			(roundrect_rratio 0.208333)
-			(net 5 "OUTDOOR_L")
+			(net 5 "/OUTDOOR_L")
 			(pintype "passive")
 		)
@@
 			(layers "F.Cu" "F.Mask" "F.Paste")
 			(roundrect_rratio 0.1)
-			(net 2 "BEACON")
+			(net 2 "/BEACON")
 			(pinfunction "DIN")
 			(pintype "input")
@@
 			(layers "F.Cu" "F.Mask" "F.Paste")
 			(roundrect_rratio 0.208333)
-			(net 6 "OUTDOOR_R")
+			(net 6 "/OUTDOOR_R")
 			(pintype "passive")
 		)
@@
 			(layers "*.Cu" "*.Mask")
 			(remove_unused_layers no)
-			(net 5 "OUTDOOR_L")
+			(net 5 "/OUTDOOR_L")
 			(pinfunction "Pin_2")
 			(pintype "passive")
@@
 			(layers "*.Cu" "*.Mask")
 			(remove_unused_layers no)
-			(net 2 "BEACON")
+			(net 2 "/BEACON")
 			(pinfunction "Pin_4")
 			(pintype "passive")
@@
 			(layers "*.Cu" "*.Mask")
 			(remove_unused_layers no)
-			(net 6 "OUTDOOR_R")
+			(net 6 "/OUTDOOR_R")
 			(pinfunction "Pin_5")
 			(pintype "passive")
 		)
-		(pad "6" thru_hole oval
+		(pad "6" thru_hole rect
 			(at 10 0)
 			(size 1.2 1.75)
@@
 	(segment
 		(start 101 66.5)
-		(end 101 59.8)
+		(end 101 61)
 		(width 0.2)
 		(layer "F.Cu")
@@
 	)
 	(segment
-		(start 101 59.8)
+		(start 102.45 59.55)
 		(end 102.45 58.35)
+		(width 0.2)
+		(layer "F.Cu")
+		(net 2)
+	)
+	(segment
+		(start 101 61)
+		(end 102.45 59.55)
 		(width 0.2)
 		(layer "F.Cu")
@@
 	)
 	(segment
-		(start 97 66.5)
-		(end 94 63.5)
+		(start 97 64)
+		(end 94 61)
 		(width 0.2)
 		(layer "F.Cu")
@@
 	)
 	(segment
-		(start 94 63.5)
+		(start 97 66.5)
+		(end 97 64)
+		(width 0.2)
+		(layer "F.Cu")
+		(net 5)
+	)
+	(segment
+		(start 94 61)
 		(end 94 59.25)
 		(width 0.2)
