File: hardware/light_board/light_board.kicad_sch (KiCad schematic)
At the start: 9 parts, among them J1 LED 1 -, J2 LED 2 -, J3 Conn_01x06_Socket, J4 LED 1 +, J5 LED 2 +

Commit message: add sponsor to PCBs
Signed-off-by: Peter Siegmund <mars3142@users.noreply.github.com>
Parts:
- D1: LCSC (none) -> 511-STM32F405RGT6; MPN (none) -> 1212
Changed lines of the file:
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@@
+			)
+		)
+		(property "MPN" "1212"
+			(at 125.73 82.55 0)
+			(effects
+				(font
+					(size 1.27 1.27)
+				)
+				(hide yes)
+			)
+		)
+		(property "LCSC" "511-STM32F405RGT6"
+			(at 125.73 82.55 0)
+			(effects
+				(font
+					(size 1.27 1.27)
+				)
+				(hide yes)
 			)
 		)
@@
 					(unit 1)
 				)
+			)
+		)
+	)
+	(symbol
+		(lib_id "pcbway:LOGO")
+		(at 190.5 106.68 0)
+		(unit 1)
+		(exclude_from_sim no)
+		(in_bom yes)
+		(on_board yes)
+		(dnp no)
+		(fields_autoplaced yes)
+		(property "Reference" "#G1"
+			(at 190.5 105.2885 0)
+			(effects
+				(font
+					(size 1.27 1.27)
+				)
+				(hide yes)
+			)
+		)
+		(property "Value" "LOGO"
+			(at 190.5 108.0715 0)
+			(effects
+				(font
+					(size 1.27 1.27)
+				)
+				(hide yes)
+			)
+		)
+		(property "Footprint" ""
+			(at 190.5 106.68 0)
+			(effects
+				(font
+					(size 1.27 1.27)
+				)
+				(hide yes)
+			)
+		)
+		(property "Datasheet" ""
+			(at 190.5 106.68 0)
+			(effects
+				(font
+					(size 1.27 1.27)
+				)
+				(hide yes)
+			)
+		)
+		(property "Description" ""
+			(at 190.5 106.68 0)
+			(effects
+				(font
+					(size 1.27 1.27)
+				)
+				(hide yes)
+			)
+		)
+		(instances
+			(project "light_board"
+				(path "/7a35f21f-dc33-4642-99a5-8943ad43e9f4"
+					(reference "#G1")
+					(unit 1)
+				)

Commit message: latest KiCad changes
Signed-off-by: Peter Siegmund <mars3142@users.noreply.github.com>
Other:
- moved on the sheet: J1, J2, J3, J4, J5, R1, R2
