File: hardware/mcu_board/mcu_board.kicad_pcb (KiCad board)
At the start: 2 copper layers, 27.2 x 54.8 mm, 12 parts, among them J1 Light, J3 Conn_ESP32-H2_Super-Mini_-_Pi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, J4 Touch, J5 Input

Commit message: latest KiCad changes
Signed-off-by: Peter Siegmund <mars3142@users.noreply.github.com>
Parts:
- removed kibuzzard-6876C010: G***, kibuzzard-6876C010
- removed kibuzzard-68B8583C: G***, kibuzzard-68B8583C
- removed kibuzzard-68C9998D: G***, kibuzzard-68C9998D
- added PS1: DB407S, aliexpress:DB407S, B.Cu at (92.6, 72.8)
- added kibuzzard-68F9205C: G***, kibuzzard-68F9205C, F.Cu at (92.0, 92.7)
- added kibuzzard-68F92064: G***, kibuzzard-68F92064, F.Cu at (97.0, 92.7)
- added kibuzzard-68F9220B: G***, kibuzzard-68F9220B, F.Cu at (111.3, 93.4)
- J3: footprint wemos:PinSocket_S3 Zero -> wemos:PinSocket_H2 Super-Mini
- renumbered J4 to J1, J1 to J2, J5 to J4, J6 to J5
Connections:
- net BEACON renamed /BEACON
- net IO renamed /IO
- net OUTDOOR_L renamed /OUTDOOR_L
- net OUTDOOR_R renamed /OUTDOOR_R
- J4 pad 1: GND -> /AC/N
- J4 pad 2: VCC -> /AC/L
Routing:
- net VCC: track 7.13 -> 17.9 mm
- net /AC/L: track 0.00 -> 10.5 mm
- net /AC/N: track 0.00 -> 10.4 mm
- net /IO: track 32.0 -> 33.0 mm
Other:
- board size 27.2 x 54.8 mm -> 28 x 54.8 mm
